Commit message: Update ARTI-H1 to the current robot and add joint system identification
- robot.urdf, agent.onnx (arti_h1 run28, 116-dim obs, outputs actions + q_des),
  292.yaml replay log (zmp02 reference) replacing the old 1000.yaml
- ARTI_H1: 116-dim observation (previous actions, gait clock), sends ONNX q_des,
  stand-up ramp to the policy default pose; robot.yaml policy section, IMU and
  sole offsets for the current robot
- motor.yaml: per-motor kp / kd (motor_command_ gains) read by MotorManager::gains(),
  measured homing offsets, homing-side limits at the stoppers
- example_sysid + config/sysid: check / step / chirp / sweep / replay tests with
  homing, safety box and abort, CSV logs for the simulator fit
- example_action: gains from motor.yaml, 2 s ramp to the first frame

Co-Authored-By: Claude Opus 5.5 <noreply@anthropic.com>

File: config/robot/ARTI-H1/robot.urdf (robot description, URDF)
Before this commit: robot robot, 16 links, 15 joints
Links:
- link left_foot: mass 0 -> 1e-9
- link left_foot_link: mass 0.13745 -> 0.15226; geometry collision mesh filename=../../meshes/arti_h1/left_foot.STL scale=0.001 0.001 0.001; visual mesh filename=../../meshes/arti_h1/left_foot.STL scale=0.001 0.001 0.001
- link left_foot_rotation: mass 0.72495 -> 0.71432; geometry collision mesh filename=../../meshes/arti_h1/left_foot_rotation.STL scale=0.001 0.001 0.001; visual mesh filename=../../meshes/arti_h1/left_foot_rotation.STL scale=0.001 0.001 0.001
- link left_hip: mass 1.1636 -> 1.13213; geometry collision mesh filename=../../meshes/arti_h1/left_hip.STL scale=0.001 0.001 0.001; visual mesh filename=../../meshes/arti_h1/left_hip.STL scale=0.001 0.001 0.001
- link left_hip_rotation: mass 0.09178 -> 0.09099; geometry collision mesh filename=../../meshes/arti_h1/left_hip_rotation.STL scale=0.001 0.001 0.001; visual mesh filename=../../meshes/arti_h1/left_hip_rotation.STL scale=0.001 0.001 0.001
- link left_shin: mass 0.59922 -> 0.58461; geometry collision mesh filename=../../meshes/arti_h1/left_shin.STL scale=0.001 0.001 0.001; visual mesh filename=../../meshes/arti_h1/left_shin.STL scale=0.001 0.001 0.001
- link left_thigh: mass 0.10518 -> 0.09972; geometry collision mesh filename=../../meshes/arti_h1/left_thigh.STL scale=0.001 0.001 0.001; visual mesh filename=../../meshes/arti_h1/left_thigh.STL scale=0.001 0.001 0.001
- link pelvis: mass 4.92214 -> 5.62607; geometry collision mesh filename=../../meshes/arti_h1/pelvis.STL scale=0.001 0.001 0.001; visual mesh filename=../../meshes/arti_h1/pelvis.STL scale=0.001 0.001 0.001
- link right_foot: mass 0 -> 1e-9
- link right_foot_link: mass 0.13745 -> 0.15226; geometry collision mesh filename=../../meshes/arti_h1/right_foot.STL scale=0.001 0.001 0.001; visual mesh filename=../../meshes/arti_h1/right_foot.STL scale=0.001 0.001 0.001
- link right_foot_rotation: mass 0.72495 -> 0.71432; geometry collision mesh filename=../../meshes/arti_h1/right_foot_rotation.STL scale=0.001 0.001 0.001; visual mesh filename=../../meshes/arti_h1/right_foot_rotation.STL scale=0.001 0.001 0.001
- link right_hip: mass 1.1636 -> 1.13213; geometry collision mesh filename=../../meshes/arti_h1/right_hip.STL scale=0.001 0.001 0.001; visual mesh filename=../../meshes/arti_h1/right_hip.STL scale=0.001 0.001 0.001
- link right_hip_rotation: mass 0.09178 -> 0.09099; geometry collision mesh filename=../../meshes/arti_h1/right_hip_rotation.STL scale=0.001 0.001 0.001; visual mesh filename=../../meshes/arti_h1/right_hip_rotation.STL scale=0.001 0.001 0.001
- link right_shin: mass 0.59922 -> 0.58461; geometry collision mesh filename=../../meshes/arti_h1/right_shin.STL scale=0.001 0.001 0.001; visual mesh filename=../../meshes/arti_h1/right_shin.STL scale=0.001 0.001 0.001
- link right_thigh: mass 0.10518 -> 0.09972; geometry collision mesh filename=../../meshes/arti_h1/right_thigh.STL scale=0.001 0.001 0.001; visual mesh filename=../../meshes/arti_h1/right_thigh.STL scale=0.001 0.001 0.001
- link trunk: mass 0 -> 1e-9
Joints:
- joint left_ankle_pitch: axis 0 -1 0 -> 0 1 0; limit lower=-2.3562 upper=0.7854 effort=100.0 velocity=5.0 -> lower=-0.7853982 upper=0.7853982 effort=24.0 velocity=5; origin xyz=0 -0.0024 -0.074 rpy=0 -0.7854 0 -> xyz=0 0.0024 -0.074 rpy=0 -0.7854 0
- joint left_ankle_roll: axis -1 0 0 -> 1 0 0; limit lower=-0.7854 upper=0.7854 effort=100.0 velocity=5.0 -> lower=-0.7853982 upper=0.7853982 effort=24.0 velocity=5; origin xyz=-0.0255 0.002 -0.060 rpy=0 0 0 -> xyz=0.0255 -0.0033 -0.06 rpy=0 0 0
- joint left_foot_frame: origin xyz=0.026 0 -0.051 rpy=0 0 0 -> xyz=-0.026 0.0 -0.051 rpy=0 0 0
- joint left_hip_pitch: axis 0 1 0 -> 0 -1 0; limit lower=-0.78 upper=1.5708 effort=100.0 velocity=30.0 -> lower=-0.7853982 upper=0.7853982 effort=23.7 velocity=30; origin xyz=0.06275 -0.0057 0 rpy=0 -0.7854 0 -> xyz=0.06275 0.0057 0.0 rpy=0 -0.7854 0
- joint left_hip_roll: limit lower=-0.34 upper=0.78 effort=100.0 velocity=30.0 -> lower=-0.7853982 upper=0.7853982 effort=23.7 velocity=30; origin xyz=-0.06325 0 -0.065 rpy=0 0 0 -> xyz=-0.06325 0.0 -0.065 rpy=0 0 0
- joint left_hip_yaw: limit lower=-0.6 upper=0.6 effort=100.0 velocity=30.0 -> lower=-0.7853982 upper=0.7853982 effort=23.7 velocity=30; origin xyz=0 0.070 -0.0066 rpy=0 0 0 -> xyz=0 0.07 0.28065 rpy=0 0 0; parent trunk -> pelvis
- joint left_knee: axis 0 1 0 -> 0 -1 0; limit lower=-1.5708 upper=0.34 effort=100.0 velocity=30.0 -> lower=-0.7853982 upper=0.7853982 effort=23.7 velocity=30; origin xyz=0 0.0114 -0.074 rpy=0 1.5708 0 -> xyz=0 -0.0114 -0.074 rpy=0 1.5708 0
- joint right_ankle_pitch: axis 0 -1 0 -> 0 1 0; limit lower=-2.3562 upper=0.7854 effort=100.0 velocity=5.0 -> lower=-0.7853982 upper=0.7853982 effort=24.0 velocity=5; origin xyz=0 -0.0024 -0.074 rpy=0 -0.7854 0 -> xyz=0 0.0024 -0.074 rpy=0 -0.7854 0
- joint right_ankle_roll: axis -1 0 0 -> 1 0 0; limit lower=-0.7854 upper=0.7854 effort=100.0 velocity=5.0 -> lower=-0.7853982 upper=0.7853982 effort=24.0 velocity=5; origin xyz=-0.0255 0.002 -0.060 rpy=0 0 0 -> xyz=0.0255 -0.0033 -0.06 rpy=0 0 0
- joint right_foot_frame: origin xyz=0.026 0 -0.051 rpy=0 0 0 -> xyz=-0.026 0.0 -0.051 rpy=0 0 0
- joint right_hip_pitch: axis 0 1 0 -> 0 -1 0; limit lower=-0.78 upper=1.5708 effort=100.0 velocity=30.0 -> lower=-0.7853982 upper=0.7853982 effort=23.7 velocity=30; origin xyz=0.06275 -0.0057 0 rpy=0 -0.7854 0 -> xyz=0.06275 0.0057 0.0 rpy=0 -0.7854 0
- joint right_hip_roll: limit lower=-0.78 upper=0.34 effort=100.0 velocity=30.0 -> lower=-0.7853982 upper=0.7853982 effort=23.7 velocity=30; origin xyz=-0.06325 0 -0.065 rpy=0 0 0 -> xyz=-0.06325 0.0 -0.065 rpy=0 0 0
- joint right_hip_yaw: limit lower=-0.6 upper=0.6 effort=100.0 velocity=30.0 -> lower=-0.7853982 upper=0.7853982 effort=23.7 velocity=30; origin xyz=0 -0.070 -0.0066 rpy=0 0 3.141592 -> xyz=0 -0.07 0.28065 rpy=0 0 3.141592; parent trunk -> pelvis
- joint right_knee: axis 0 1 0 -> 0 -1 0; limit lower=-1.5708 upper=0.34 effort=100.0 velocity=30.0 -> lower=-0.7853982 upper=0.7853982 effort=23.7 velocity=30; origin xyz=0 0.0114 -0.074 rpy=0 1.5708 0 -> xyz=0 -0.0114 -0.074 rpy=0 1.5708 0
- joint trunk_frame: origin xyz=0 0 0.29525 rpy=0 0 0 -> xyz=0 0 0.28725 rpy=0 0 0
